File: Hardware/Rudolph_Tracker/Rudolph_Tracker.kicad_pcb (KiCad board)
At the start: 4 copper layers, 45.6 x 25 mm, 57 parts, among them J1 SOICbite, J2 USB_C_Receptacle_USB2.0, J3 537480208, J4 U.FL, J5 537480208, Q1 IRLML0060TRPBF, U1 RP2040, U4 W25Q128JVS, U7 MS5607-02BA, U8 DRF1262TL, Y1 445I23D12M00000, Y2 32.768k

Commit message: generating gerbers
Changed lines of the file:
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@@
       (plot_on_all_layers_selection 0x0000000_00000000)
       (disableapertmacros false)
-      (usegerberextensions false)
-      (usegerberattributes true)
-      (usegerberadvancedattributes true)
-      (creategerberjobfile true)
+      (usegerberextensions true)
+      (usegerberattributes false)
+      (usegerberadvancedattributes false)
+      (creategerberjobfile false)
       (dashed_line_dash_ratio 12.000000)
       (dashed_line_gap_ratio 3.000000)
@@
       (psa4output false)
       (plotreference true)
-      (plotvalue true)
+      (plotvalue false)
       (plotinvisibletext false)
       (sketchpadsonfab false)
-      (subtractmaskfromsilk false)
+      (subtractmaskfromsilk true)
       (outputformat 1)
       (mirror false)
-      (drillshape 1)
+      (drillshape 0)
       (scaleselection 1)
-      (outputdirectory "")
+      (outputdirectory "Gerber/")
     )
   )
@@
     (fp_line (start 3.5 3.5) (end -3.5 3.5)
       (stroke (width 0.1) (type solid)) (layer "F.Fab"))
-    (pad "" smd roundrect (at -0.6375 -0.6375 90) (size 1.084435 1.084435) (layers "F.Paste") (roundrect_rratio 0.230535))
-    (pad "" smd roundrect (at -0.6375 0.6375 90) (size 1.084435 1.084435) (layers "F.Paste") (roundrect_rratio 0.230535))
-    (pad "" smd roundrect (at 0.6375 -0.6375 90) (size 1.084435 1.084435) (layers "F.Paste") (roundrect_rratio 0.230535))
-    (pad "" smd roundrect (at 0.6375 0.6375 90) (size 1.084435 1.084435) (layers "F.Paste") (roundrect_rratio 0.230535))
+    (pad "" smd roundrect (at -0.6375 -0.6375 90) (size 1.084435 1.084435) (layers "F.Paste") (roundrect_rratio 0.2305347946))
+    (pad "" smd roundrect (at -0.6375 0.6375 90) (size 1.084435 1.084435) (layers "F.Paste") (roundrect_rratio 0.2305347946))
+    (pad "" smd roundrect (at 0.6375 -0.6375 90) (size 1.084435 1.084435) (layers "F.Paste") (roundrect_rratio 0.2305347946))
+    (pad "" smd roundrect (at 0.6375 0.6375 90) (size 1.084435 1.084435) (layers "F.Paste") (roundrect_rratio 0.2305347946))
     (pad "1" smd roundrect (at -3.4375 -2.6 90) (size 0.875 0.2) (layers "F.Cu" "F.Paste" "F.Mask") (roundrect_rratio 0.25)
       (net 7 "+3V3") (pinfunction "IOVDD") (pintype "power_in"))
@@
     (property "ki_keywords" "537480208")
     (attr smd)
-    (fp_text reference "J3" (at -5.3 -3.4 90 unlocked) (layer "F.SilkS")
+    (fp_text reference "J3" (at -4.75 -3.5 unlocked) (layer "F.SilkS")
         (effects (font (size 1 1) (thickness 0.15)))
     )
@@
     (pad "20" smd rect (at 2.250001 1.700002 90) (size 0.25 1.2) (layers "F.Cu" "F.Paste" "F.Mask")
       (net 1 "GND") (pinfunction "20") (pintype "unspecified"))
+    (model "/Users/michaelshipman/Downloads/537480208.stp"
+      (offset (xyz 0 0 1.2))
+      (scale (xyz 1 1 1))
+      (rotate (xyz -90 0 0))
+    )
   )
   (footprint "Capacitor_SMD:C_0402_1005Metric" (layer "F.Cu")
@@
     (property "ki_keywords" "537480208")
     (attr smd)
-    (fp_text reference "J5" (at -6 -2.1 90 unlocked) (layer "F.SilkS")
+    (fp_text reference "J5" (at -6 -2.25 unlocked) (layer "F.SilkS")
         (effects (font (size 1 1) (thickness 0.15)))
     )
@@
     (pad "20" smd rect (at 2.250001 1.700002 90) (size 0.25 1.2) (layers "F.Cu" "F.Paste" "F.Mask")
       (net 1 "GND") (pinfunction "20") (pintype "unspecified"))
+    (model "/Users/michaelshipman/Downloads/537480208.stp"
+      (offset (xyz 0 0 1.2))
+      (scale (xyz 1 1 1))
+      (rotate (xyz -90 0 0))
+    )
   )
   (footprint "Capacitor_SMD:C_0402_1005Metric" (layer "F.Cu")

Commit message: generating some BOMs
Routing:
- net /QSPI_SS: track 25.2 -> 24.6 mm
Changed lines of the file:
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@@
   (segment (start 87.5 117.7) (end 85.41 117.7) (width 0.286) (layer "F.Cu") (net 23))
   (segment (start 86.8 130.1) (end 83.995 130.1) (width 0.2) (layer "F.Cu") (net 24))
-  (segment (start 87.1 130.4) (end 95 130.4) (width 0.2) (layer "F.Cu") (net 24))
   (segment (start 88.2 129.2) (end 87.3 130.1) (width 0.2) (layer "F.Cu") (net 24))
+  (segment (start 95.89 129.51) (end 95.89 128.9) (width 0.2) (layer "F.Cu") (net 24))
+  (segment (start 87.3 130.1) (end 87.4 130.2) (width 0.2) (layer "F.Cu") (net 24))
   (segment (start 88.2 123.1625) (end 88.2 129.2) (width 0.2) (layer "F.Cu") (net 24))
   (segment (start 89.0625 122.3) (end 88.2 123.1625) (width 0.2) (layer "F.Cu") (net 24))
-  (segment (start 86.8 130.1) (end 87.1 130.4) (width 0.2) (layer "F.Cu") (net 24))
-  (segment (start 95.89 129.51) (end 95.89 128.9) (width 0.2) (layer "F.Cu") (net 24))
-  (segment (start 95 130.4) (end 95.89 129.51) (width 0.2) (layer "F.Cu") (net 24))
+  (segment (start 95.2 130.2) (end 95.89 129.51) (width 0.2) (layer "F.Cu") (net 24))
+  (segment (start 87.4 130.2) (end 95.2 130.2) (width 0.2) (layer "F.Cu") (net 24))
   (segment (start 87.3 130.1) (end 86.8 130.1) (width 0.2) (layer "F.Cu") (net 24))
   (segment (start 83.995 130.1) (end 82.495 128.6) (width 0.2) (layer "F.Cu") (net 24))
