File: Hardware/Rudolph_Tracker/Rudolph_Tracker.kicad_sch (KiCad schematic)
At the start: 57 parts, among them J1 USB_C_Receptacle_USB2.0, J2 SOICbite, J3 537480208, J4 U.FL, J5 537480208, Q1 IRLML0060TRPBF, U2 RP2040, U3 W25Q128JVS, U6 MS5607-02BA, U8 DRF1262TL, Y1 445I23D12M00000, Y2 32.768k

Commit message: generating gerbers
Parts:
- J3, J5: value 537480208 -> 0539160208
Other:
- note added: "Technically the footprint used here is for a slightly different but pin compatible part. The only difference is mating height which needs to be greater than 3.31mm to account for the USB connector."
Changed lines of the file:
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@@
     (effects (font (size 5.08 5.08) (thickness 1.016) bold) (justify left bottom))
+  )
+  (text "Technically the footprint used here is for \na slightly different but pin compatible part.\nThe only difference is mating height which needs\nto be greater than 3.31mm to account for the USB connector."
+    (at 209.55 209.55 0)
+    (effects (font (size 1.27 1.27)) (justify left bottom))
   )
   (text "GPS" (at 273.05 71.12 0)
@@
       (effects (font (size 1.524 1.524)))
     )
-    (property "Value" "537480208" (at 198.12 196.85 0)
+    (property "Value" "0539160208" (at 198.12 196.85 0)
       (effects (font (size 1.524 1.524)))
     )
@@
       (effects (font (size 1.524 1.524)))
     )
-    (property "Value" "537480208" (at 157.48 196.85 0)
+    (property "Value" "0539160208" (at 157.48 196.85 0)
       (effects (font (size 1.524 1.524)))
     )

Commit message: generating some BOMs
Parts:
- R21, R22: value 33 -> 0
- U3: value W25Q128JVS -> W25Q64JVZP
Changed lines of the file:
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@@
       (effects (font (size 1.27 1.27)))
     )
-    (property "Value" "33" (at 220.98 55.88 90)
+    (property "Value" "0" (at 220.98 55.88 90)
       (effects (font (size 0.8 0.8)))
     )
@@
       (effects (font (size 1.27 1.27)))
     )
-    (property "Value" "W25Q128JVS" (at 176.53 127 0)
+    (property "Value" "W25Q64JVZP" (at 176.53 127 0)
       (effects (font (size 1.27 1.27)))
     )
@@
       (effects (font (size 1.27 1.27)))
     )
-    (property "Value" "33" (at 220.98 53.34 90)
+    (property "Value" "0" (at 220.98 53.34 90)
       (effects (font (size 0.8 0.8)))
     )

Commit message: messing with libraries
Other:
- company: (none) -> BPP
- title: (none) -> Rudolph Tracker
Changed lines of the file:
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@@
 (kicad_sch (version 20230121) (generator eeschema)
   (paper "A3")
+  (title_block
+    (title "Rudolph Tracker")
+    (date "2023-10-18")
+    (rev "V0.0")
+    (company "BPP")
+    (comment 1 "Michael Shipman")
+  )
   (junction (at 100.33 21.59) (diameter 0) (color 0 0 0 0)
   )
