File: Hardware/PowerPack/PowerPack.kicad_sch (KiCad schematic)
At the start: 51 parts, among them J2 529910208, J3 529910208, J4 XT30, U10 TPS2121RUXR, U5 MAX25232ATCB/V+T, U7 LT6703CDC-3, U8 MAX77857

Commit message: messing with libraries
Other:
- company: (none) -> BPP
- title: (none) -> PowerPack
Changed lines of the file:
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@@
 (kicad_sch (version 20230121) (generator eeschema)
   (paper "A4")
+  (title_block
+    (title "PowerPack")
+    (date "2023-10-18")
+    (rev "V0.0")
+    (company "BPP")
+    (comment 1 "Michael Shipman")
+  )
   (junction (at 123.19 105.41) (diameter 0) (color 0 0 0 0)
   )
